Commit message: Trying to fix URDF

File: urdf/barbot_test.urdf (robot description, URDF)
Before this commit: robot barbot_test, 6 links, 5 joints
Links:
- added link world
- link link1: geometry visual mesh filename=package://bar-bot/mesh/Link0.STL scale=0.001 0.001 0.001
- link link2: geometry visual mesh filename=package://bar-bot/mesh/Link1.STL scale=0.001 0.001 0.001
- link link3: geometry visual mesh filename=package://bar-bot/mesh/Link2.STL scale=0.001 0.001 0.001
- link link4: geometry visual mesh filename=package://bar-bot/mesh/Link3.STL scale=0.001 0.001 0.001
- link link5: geometry visual mesh filename=package://bar-bot/mesh/Link4_5.STL scale=0.001 0.001 0.001
- link link6: geometry visual mesh filename=package://bar-bot/mesh/Link4_5.STL scale=0.001 0.001 0.001
Joints:
- added joint world_joint: type fixed, parent world, child link1, origin xyz=0 0 0 rpy=0 0 0, axis 0 0 1
- joint joint1: origin xyz=0 0 31.1 rpy=0 0 0 -> xyz=0 0 0.0311 rpy=0 0 0; parent link1 -> world
- joint joint2: origin xyz=61.1 0 50 rpy=0 1.570796 -0.78539816 -> xyz=0.0611 0 0.050 rpy=0 -1.570796 -0.78539816; parent link2 -> world
- joint joint3: origin xyz=155.56 0 -31.1 rpy=3.1415926 0 -1.570796 -> xyz=0.15556 0 -0.0311 rpy=3.1415926 0 -1.570796
- joint joint4: origin xyz=142.42 0 -31.1 rpy=3.1415926 0 -0.78539816 -> xyz=0.14142 0 -0.0311 rpy=3.1415926 0 -0.78539816
- joint joint5: origin xyz=81.1 0 0 rpy=0 0 0 -> xyz=0.0811 0 0 rpy=0 0 0
