Commit message: End of last friday commit - ikin broken

File: urdf/solidworks-bar-bot.urdf (robot description, URDF)
Before this commit: robot _BarBot.SLDASM, 6 links, 5 joints
Links:
- removed link base_link
- removed link link_grippy
- added link dummy; visual box size=0.2 0.2 0.0254
- added link link_5, mass 0.196644768; collision mesh filename=package://bar-bot/mesh/link_5.STL; visual mesh filename=package://bar-bot/mesh/link_5.STL
- added link world, mass 0.250135388974212; collision mesh filename=package://bar-bot/mesh/base_link.STL; visual mesh filename=package://bar-bot/mesh/base_link.STL
- link link_2: mass 0.147378954309203 -> 0.611278584185544
- link link_3: mass 0.137479459372592 -> 0.369429274310776
- link link_4: mass 0.104469603548198 -> 0.336419418486383
Joints:
- added joint joint_tip: type continuous, parent link_5, child dummy, origin xyz=0 0 0.1128 rpy=0 0 0, axis 0 0 1
- joint joint_1: axis 0 -5.7223E-05 -1 -> 0 0 1; limit lower=-3.14 upper=3.14 effort=0 velocity=0 -> (none); origin xyz=0 -0.0361 0 rpy=1.5709 -6.1234E-17 -1.5708 -> xyz=0 -0.0361 0 rpy=0 0 -1.5707963267949; parent base_link -> world
- joint joint_2: axis 0.67783 0.73522 0 -> 0 0 1; limit lower=-3.14 upper=3.14 effort=0 velocity=0 -> (none); origin xyz=0.049993 0.00059543 -0.0611 rpy=3.1415 8.4143E-05 0.82599 -> xyz=0.05 0 -0.0611 rpy=-3.14159265358979 0 1.5707963267949
- joint joint_3: axis -0.73542 -0.67762 0 -> 0 0 1; limit lower=-3.14 upper=3.14 effort=0 velocity=0 -> (none); origin xyz=0.15513 0.00041367 -0.0311 rpy=3.1416 8.6407E-16 -1.5711 -> xyz=0.155563491861 0 -0.0311 rpy=0 0 0
- joint joint_4: axis 0.99993 5.7223E-05 0.012049 -> 0 1 0; limit lower=-3.14 upper=3.14 effort=0 velocity=0 -> (none); origin xyz=0.14142 0 -0.0311 rpy=1.5708 1.623E-15 -0.81423 -> xyz=0.141421356237 0 0.0311 rpy=-1.57079632679489 0 -0.0120495748569734
- joint joint_5: axis -0.15792 -0.98738 -0.012049 -> 0 0 1; child link_grippy -> link_5; limit lower=-3.14 upper=3.14 effort=0 velocity=0 -> (none); origin xyz=0.0811 0.0561 0 rpy=-1.5708 0.15859 -1.5708 -> xyz=0.0810882254780547 0.0560999999999999 0.000977125933747033 rpy=1.57079632679489 0.0653055782012251 1.5707963267949
