Commit message: ikin, urdf, and HebiHelper now work!

File: urdf/basic_arm.urdf (robot description, URDF)
Before this commit: robot myrobot, 7 links, 6 joints
Joints:
- joint pitch_1: origin xyz=0 0 0.0861 rpy=0 0 0 -> xyz=0 0 .106 rpy=0 0 0
- joint pitch_2: axis 1 0 0 -> -1 0 0; origin xyz=0 .15556 0 rpy=0 0 0 -> xyz=0 .16 0 rpy=0 0 0
- joint pitch_3: origin xyz=0 .14142 0 rpy=0 0 0 -> xyz=0 .16 0 rpy=0 0 0
- joint yaw: origin xyz=0 .1827 0 rpy=0 0 0 -> xyz=0 .16 0 rpy=0 0 0

Commit message: Trajectories work!

File: urdf/basic_arm.urdf (robot description, URDF)
Before this commit: robot myrobot, 7 links, 6 joints
Joints:
- joint pitch_2: axis -1 0 0 -> 1 0 0
